Commit message: update control and set limits

File: playground/public/URDF/so_arm100.urdf (robot description, URDF)
Before this commit: robot so_arm100, 7 links, 6 joints
Joints:
- joint Elbow: limit lower=0 upper=3.14158 effort=35 velocity=1 -> lower=-3.14158 upper=0 effort=35 velocity=1
- joint Pitch: limit lower=-3.14158 upper=0.2 effort=35 velocity=1 -> lower=0 upper=3.5 effort=35 velocity=1
- joint Rotation: limit lower=-2.2 upper=2.2 effort=35 velocity=1 -> lower=-2 upper=2 effort=35 velocity=1
- joint Wrist_Pitch: limit lower=-2.0 upper=1.8 effort=35 velocity=1 -> lower=-2.5 upper=1.2 effort=35 velocity=1
