Commit message: bambot urdf without wheels

File: playground/public/URDF/bambot.urdf (robot description, URDF)
Before this commit: robot so_arm100, 7 links, 6 joints
Links:
- removed link Base
- removed link Fixed_Jaw
- removed link Lower_Arm
- removed link Moving_Jaw
- removed link Rotation_Pitch
- removed link Upper_Arm
- removed link Wrist_Pitch_Roll
- added link base_link; visual mesh filename=meshes/Bambot_Body.stl scale=0.001 0.001 0.001
- added link left_arm_Base, mass 1.0; collision mesh filename=meshes/Base.stl; visual mesh filename=meshes/Base.stl
- added link left_arm_Fixed_Jaw, mass 0.0929859; visual mesh filename=meshes/Fixed_Jaw.stl; visual mesh filename=meshes/Fixed_Jaw_Motor.stl
- added link left_arm_Lower_Arm, mass 0.147968; collision mesh filename=meshes/Lower_Arm.stl; visual mesh filename=meshes/Lower_Arm.stl
- added link left_arm_Moving_Jaw, mass 0.0202444; visual mesh filename=meshes/Moving_Jaw.stl
- added link left_arm_Rotation_Pitch, mass 0.119226; collision mesh filename=meshes/Rotation_Pitch.stl; visual mesh filename=meshes/Rotation_Pitch.stl
- added link left_arm_Upper_Arm, mass 0.162409; collision mesh filename=meshes/Upper_Arm.stl; visual mesh filename=meshes/Upper_Arm.stl
- added link left_arm_Wrist_Pitch_Roll, mass 0.0661321; collision mesh filename=meshes/Wrist_Pitch_Roll.stl; visual mesh filename=meshes/Wrist_Pitch_Roll.stl
- added link right_arm_Base, mass 1.0; collision mesh filename=meshes/Base.stl; visual mesh filename=meshes/Base.stl
- added link right_arm_Fixed_Jaw, mass 0.0929859; visual mesh filename=meshes/Fixed_Jaw.stl; visual mesh filename=meshes/Fixed_Jaw_Motor.stl
- added link right_arm_Lower_Arm, mass 0.147968; collision mesh filename=meshes/Lower_Arm.stl; visual mesh filename=meshes/Lower_Arm.stl
- added link right_arm_Moving_Jaw, mass 0.0202444; visual mesh filename=meshes/Moving_Jaw.stl
- added link right_arm_Rotation_Pitch, mass 0.119226; collision mesh filename=meshes/Rotation_Pitch.stl; visual mesh filename=meshes/Rotation_Pitch.stl
- added link right_arm_Upper_Arm, mass 0.162409; collision mesh filename=meshes/Upper_Arm.stl; visual mesh filename=meshes/Upper_Arm.stl
- added link right_arm_Wrist_Pitch_Roll, mass 0.0661321; collision mesh filename=meshes/Wrist_Pitch_Roll.stl; visual mesh filename=meshes/Wrist_Pitch_Roll.stl
Joints:
- removed joint Elbow
- removed joint Jaw
- removed joint Pitch
- removed joint Rotation
- removed joint Wrist_Pitch
- removed joint Wrist_Roll
- added joint left_arm_Elbow: type revolute, parent left_arm_Upper_Arm, child left_arm_Lower_Arm, origin xyz=0 0.11257 0.028 rpy=-1.57079 0 0, axis 1 0 0, limit lower=-3.14158 upper=0 effort=35 velocity=1
- added joint left_arm_Jaw: type revolute, parent left_arm_Fixed_Jaw, child left_arm_Moving_Jaw, origin xyz=-0.0202 -0.0244 0 rpy=0 3.14158 0, axis 0 0 1, limit lower=-0.2 upper=2.0 effort=35 velocity=1
- added joint left_arm_Pitch: type revolute, parent left_arm_Rotation_Pitch, child left_arm_Upper_Arm, origin xyz=0 0.1025 0.0306 rpy=-0.1 0 0, axis 1 0 0, limit lower=0 upper=3.5 effort=35 velocity=1
- added joint left_arm_Rotation: type revolute, parent left_arm_Base, child left_arm_Rotation_Pitch, origin xyz=0 -0.0452 0.0165 rpy=1.57079 0 0, axis 0 1 0, limit lower=-2 upper=2 effort=35 velocity=1
- added joint left_arm_Wrist_Pitch: type revolute, parent left_arm_Lower_Arm, child left_arm_Wrist_Pitch_Roll, origin xyz=0 0.0052 0.1349 rpy=-1.57079 0 0, axis 1 0 0, limit lower=-2.5 upper=1.2 effort=35 velocity=1
- added joint left_arm_Wrist_Roll: type revolute, parent left_arm_Wrist_Pitch_Roll, child left_arm_Fixed_Jaw, origin xyz=0 -0.0601 0 rpy=0 0 0, axis 0 1 0, limit lower=-3.14158 upper=3.14158 effort=35 velocity=1
- added joint left_arm_to_base: type fixed, parent base_link, child left_arm_Base, origin xyz=-0.18 -0.07 0.64 rpy=0 3.14158 1.5708
- added joint right_arm_Elbow: type revolute, parent right_arm_Upper_Arm, child right_arm_Lower_Arm, origin xyz=0 0.11257 0.028 rpy=-1.57079 0 0, axis 1 0 0, limit lower=-3.14158 upper=0 effort=35 velocity=1
- added joint right_arm_Jaw: type revolute, parent right_arm_Fixed_Jaw, child right_arm_Moving_Jaw, origin xyz=-0.0202 -0.0244 0 rpy=0 3.14158 0, axis 0 0 1, limit lower=-0.2 upper=2.0 effort=35 velocity=1
- added joint right_arm_Pitch: type revolute, parent right_arm_Rotation_Pitch, child right_arm_Upper_Arm, origin xyz=0 0.1025 0.0306 rpy=-0.1 0 0, axis 1 0 0, limit lower=0 upper=3.5 effort=35 velocity=1
- added joint right_arm_Rotation: type revolute, parent right_arm_Base, child right_arm_Rotation_Pitch, origin xyz=0 -0.0452 0.0165 rpy=1.57079 0 0, axis 0 1 0, limit lower=-2 upper=2 effort=35 velocity=1
- added joint right_arm_Wrist_Pitch: type revolute, parent right_arm_Lower_Arm, child right_arm_Wrist_Pitch_Roll, origin xyz=0 0.0052 0.1349 rpy=-1.57079 0 0, axis 1 0 0, limit lower=-2.5 upper=1.2 effort=35 velocity=1
- added joint right_arm_Wrist_Roll: type revolute, parent right_arm_Wrist_Pitch_Roll, child right_arm_Fixed_Jaw, origin xyz=0 -0.0601 0 rpy=0 0 0, axis 0 1 0, limit lower=-3.14158 upper=3.14158 effort=35 velocity=1
- added joint right_arm_to_base: type fixed, parent base_link, child right_arm_Base, origin xyz=-0.17 -0.42 0.64 rpy=0 3.14158 1.5708

Commit message: init bot swith

File: playground/public/URDF/bambot.urdf (robot description, URDF)
Before this commit: robot bambot, 15 links, 14 joints
Links:
- added link front_left_wheel, mass 1.0; collision cylinder length=0.05 radius=0.075; visual mesh filename=meshes/BambotWheel.stl scale=0.001 0.001 0.001
- added link front_right_wheel, mass 1.0; collision cylinder length=0.05 radius=0.075; visual mesh filename=meshes/BambotWheel.stl scale=0.001 0.001 0.001
- added link rear_wheel, mass 1.0; collision cylinder length=0.05 radius=0.075; visual mesh filename=meshes/BambotWheel.stl scale=0.001 0.001 0.001
Joints:
- added joint front_left_wheel_joint: type continuous, parent base_link, child front_left_wheel, origin xyz=-0.1 0.0 -0.03 rpy=0 1.5708 -2.0944, axis 0 1 0
- added joint front_right_wheel_joint: type continuous, parent base_link, child front_right_wheel, origin xyz=-0.1 -0.48 -0.03 rpy=0 1.5708 2.0944, axis 0 1 0
- added joint rear_wheel_joint: type continuous, parent base_link, child rear_wheel, origin xyz=-0.52 -0.25 -0.03 rpy=0 1.5708 0, axis 0 1 0

Commit message: update joint limits

File: playground/public/URDF/bambot.urdf (robot description, URDF)
Before this commit: robot bambot, 18 links, 17 joints
Joints:
- joint left_arm_Elbow: limit lower=-3.14158 upper=0 effort=35 velocity=1 -> lower=0 upper=3 effort=35 velocity=1
- joint left_arm_Jaw: limit lower=-0.2 upper=2.0 effort=35 velocity=1 -> lower=-0.2 upper=1.7 effort=35 velocity=1
- joint left_arm_Pitch: limit lower=0 upper=3.5 effort=35 velocity=1 -> lower=-1.4 upper=1.7139 effort=35 velocity=1
- joint left_arm_Wrist_Pitch: limit lower=-2.5 upper=1.2 effort=35 velocity=1 -> lower=-1.8 upper=1.8 effort=35 velocity=1
- joint left_arm_Wrist_Roll: limit lower=-3.14158 upper=3.14158 effort=35 velocity=1 -> lower=-1.57079 upper=1.57079 effort=35 velocity=1
- joint right_arm_Elbow: limit lower=-3.14158 upper=0 effort=35 velocity=1 -> lower=0 upper=3 effort=35 velocity=1
- joint right_arm_Jaw: limit lower=-0.2 upper=2.0 effort=35 velocity=1 -> lower=-0.2 upper=1.7 effort=35 velocity=1
- joint right_arm_Pitch: limit lower=0 upper=3.5 effort=35 velocity=1 -> lower=-1.4 upper=1.7139 effort=35 velocity=1
- joint right_arm_Wrist_Pitch: limit lower=-2.5 upper=1.2 effort=35 velocity=1 -> lower=-1.8 upper=1.8 effort=35 velocity=1
- joint right_arm_Wrist_Roll: limit lower=-3.14158 upper=3.14158 effort=35 velocity=1 -> lower=-1.57079 upper=1.57079 effort=35 velocity=1

Commit message: keyboard control v0

File: playground/public/URDF/bambot.urdf (robot description, URDF)
Before this commit: robot bambot, 18 links, 17 joints
Joints:
- joint front_left_wheel_joint: axis 0 1 0 -> 0 0 1
- joint front_right_wheel_joint: axis 0 1 0 -> 0 0 1
- joint rear_wheel_joint: axis 0 1 0 -> 0 0 1
