Commit message: update urdf default angle

File: website/public/URDF/so_arm100.urdf (robot description, URDF)
Before this commit: robot so_arm100, 7 links, 6 joints
Joints:
- joint Jaw: limit lower=-0.2 upper=2.0 effort=35 velocity=1 -> lower=-0.03 upper=2.0 effort=35 velocity=1; origin xyz=-0.0202 -0.0244 0 rpy=0 3.14158 0 -> xyz=-0.0202 -0.0244 0 rpy=0 3.14158 0.17
- joint Wrist_Pitch: limit lower=-2.5 upper=1.2 effort=35 velocity=1 -> lower=-2.6 upper=0.5 effort=35 velocity=1; origin xyz=0 0.0052 0.1349 rpy=-1 0 0 -> xyz=0 0.0052 0.1349 rpy=-0.5 0 0
